File: hw/traincontrol-shield/rail-voltage-sense.kicad_sch (KiCad schematic)
At the start: 2 parts

Commit message: Fix schematic ERC errors: pin Y-flip, PWR_FLAG, label wiring, spacing
- Fix connector pin positions using Y-flip convention (sym Y-up → sch Y-down)
- Add GND PWR_FLAG to power-supply sheet (eliminates power_pin_not_driven)
- Fix top-level connector label placement: labels at stub end, wires toward pins
- Apply omnidirectional spacing and IC-to-passive body gap rules across sheets
- Update schematics-plan.md with ERC workflow and coordinate conventions
- Regenerate all sub-sheets with corrected generator scripts

ERC result: 138 violations (all warnings/cosmetic), 0 critical errors.

Co-Authored-By: Claude Opus 4.6 <noreply@anthropic.com>
Changed lines of the file:
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@@
 	)
 	(wire
-		(pts (xy 80.01 80.01) (xy 80.01 87.63))
+		(pts (xy 80.01 80.01) (xy 80.01 83.82))
 		(stroke (width 0) (type solid))
 	)
+	(wire
+		(pts (xy 80.01 83.82) (xy 80.01 87.63))
+		(stroke (width 0) (type solid))
+	)
