File: hw/traincontrol-shield/mcu.kicad_sch (KiCad schematic)
At the start: 18 parts, among them CON5 ConnectionPad, CON6 ConnectionPad, CON7 ConnectionPad, SW1 SW_Push, SW2 SW_Push, U7 ESP32-C3-MINI-1-N4

Commit message: Update BOM, docs, and JLCPCB outputs to match current schematics
- Update BOM.md with JLCPCB LCSC part numbers for all components
- Generate JLCPCB BOM and CPL files for PCBA ordering
- Update docs and README to reflect component changes (BAT54S/SS34
  rectification, BT134W-600E TRIACs, EL357N optocoupler, ESP32-C3)
- Suppress ERC warnings for unspecified pin connections in project settings

Co-Authored-By: Claude Opus 4.6 <noreply@anthropic.com>
Parts:
- SW1, SW2: now not fitted; now left out of the parts list
Changed lines of the file:
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@@
 		(unit 1)
 		(exclude_from_sim no)
-		(in_bom yes)
-		(on_board yes)
-		(dnp no)
+		(in_bom no)
+		(on_board yes)
+		(dnp yes)
 		(property "Reference" "SW2"
 			(at 238.76 89.408 0)
@@
 				(path "/12cc2a67-9b1c-41e4-828f-9c2a8df6bb35/8c6fba78-5fd4-419a-8456-de6c668aaabc"
 					(reference "SW2")
+					(unit 1)
+				)
+			)
+			(project "mcu"
+				(path "/b17ddd41-b910-4f09-a62f-46566a666def"
+					(reference "SW?")
 					(unit 1)
 				)
@@
 				)
 			)
+			(project "mcu"
+				(path "/b17ddd41-b910-4f09-a62f-46566a666def"
+					(reference "R?")
+					(unit 1)
+				)
+			)
 		)
 	)
@@
 		(unit 1)
 		(exclude_from_sim no)
-		(in_bom yes)
-		(on_board yes)
-		(dnp no)
+		(in_bom no)
+		(on_board yes)
+		(dnp yes)
 		(property "Reference" "SW1"
 			(at 239.014 56.642 0)
@@
 				)
 			)
+			(project "mcu"
+				(path "/b17ddd41-b910-4f09-a62f-46566a666def"
+					(reference "SW?")
+					(unit 1)
+				)
+			)
 		)
 	)
@@
 				)
 			)
+			(project "mcu"
+				(path "/b17ddd41-b910-4f09-a62f-46566a666def"
+					(reference "#PWR?")
+					(unit 1)
+				)
+			)
 		)
 	)
@@
 				(path "/12cc2a67-9b1c-41e4-828f-9c2a8df6bb35/8c6fba78-5fd4-419a-8456-de6c668aaabc"
 					(reference "#PWR08")
+					(unit 1)
+				)
+			)
+			(project "mcu"
+				(path "/b17ddd41-b910-4f09-a62f-46566a666def"
+					(reference "#PWR?")
 					(unit 1)
 				)
@@
 				)
 			)
+			(project "mcu"
+				(path "/b17ddd41-b910-4f09-a62f-46566a666def"
+					(reference "R?")
+					(unit 1)
+				)
+			)
 		)
 	)
@@
 				)
 			)
+			(project "mcu"
+				(path "/b17ddd41-b910-4f09-a62f-46566a666def"
+					(reference "R?")
+					(unit 1)
+				)
+			)
 		)
 	)
@@
 				)
 			)
+			(project "mcu"
+				(path "/b17ddd41-b910-4f09-a62f-46566a666def"
+					(reference "#PWR?")
+					(unit 1)
+				)
+			)
 		)
 	)
@@
 				)
 			)
+			(project "mcu"
+				(path "/b17ddd41-b910-4f09-a62f-46566a666def"
+					(reference "CON?")
+					(unit 1)
+				)
+			)
 		)
 	)
@@
 				)
 			)
+			(project "mcu"
+				(path "/b17ddd41-b910-4f09-a62f-46566a666def"
+					(reference "R?")
+					(unit 1)
+				)
+			)
 		)
 	)
@@
 				)
 			)
+			(project "mcu"
+				(path "/b17ddd41-b910-4f09-a62f-46566a666def"
+					(reference "#PWR?")
+					(unit 1)
+				)
+			)
 		)
 	)
@@
 				)
 			)
+			(project "mcu"
+				(path "/b17ddd41-b910-4f09-a62f-46566a666def"
+					(reference "U?")
+					(unit 1)
+				)
+			)
 		)
 	)
@@
 				(path "/12cc2a67-9b1c-41e4-828f-9c2a8df6bb35/8c6fba78-5fd4-419a-8456-de6c668aaabc"
 					(reference "C12")
+					(unit 1)
+				)
+			)
+			(project "mcu"
+				(path "/b17ddd41-b910-4f09-a62f-46566a666def"
+					(reference "C?")
 					(unit 1)
 				)
@@
 				)
 			)
+			(project "mcu"
+				(path "/b17ddd41-b910-4f09-a62f-46566a666def"
+					(reference "#PWR?")
+					(unit 1)
+				)
+			)
 		)
 	)
@@
 				(path "/12cc2a67-9b1c-41e4-828f-9c2a8df6bb35/8c6fba78-5fd4-419a-8456-de6c668aaabc"
 					(reference "D4")
+					(unit 1)
+				)
+			)
+			(project "mcu"
+				(path "/b17ddd41-b910-4f09-a62f-46566a666def"
+					(reference "D?")
 					(unit 1)
 				)
@@
 				)
 			)
+			(project "mcu"
+				(path "/b17ddd41-b910-4f09-a62f-46566a666def"
+					(reference "#PWR?")
+					(unit 1)
+				)
+			)
 		)
 	)
@@
 				)
 			)
+			(project "mcu"
+				(path "/b17ddd41-b910-4f09-a62f-46566a666def"
+					(reference "#PWR?")
+					(unit 1)
+				)
+			)
 		)
 	)
@@
 				)
 			)
+			(project "mcu"
+				(path "/b17ddd41-b910-4f09-a62f-46566a666def"
+					(reference "R?")
+					(unit 1)
+				)
+			)
 		)
 	)
@@
 				)
 			)
+			(project "mcu"
+				(path "/b17ddd41-b910-4f09-a62f-46566a666def"
+					(reference "#PWR?")
+					(unit 1)
+				)
+			)
 		)
 	)
@@
 				)
 			)
+			(project "mcu"
+				(path "/b17ddd41-b910-4f09-a62f-46566a666def"
+					(reference "R?")
+					(unit 1)
+				)
+			)
 		)
 	)
@@
 				)
 			)
+			(project "mcu"
+				(path "/b17ddd41-b910-4f09-a62f-46566a666def"
+					(reference "#PWR?")
+					(unit 1)
+				)
+			)
 		)
 	)
@@
 				)
 			)
+			(project "mcu"
+				(path "/b17ddd41-b910-4f09-a62f-46566a666def"
+					(reference "R?")
+					(unit 1)
+				)
+			)
 		)
 	)
@@
 				)
 			)
+			(project "mcu"
+				(path "/b17ddd41-b910-4f09-a62f-46566a666def"
+					(reference "CON?")
+					(unit 1)
+				)
+			)
 		)
 	)
@@
 				)
 			)
+			(project "mcu"
+				(path "/b17ddd41-b910-4f09-a62f-46566a666def"
+					(reference "#PWR?")
+					(unit 1)
+				)
+			)
 		)
 	)
@@
 				)
 			)
+			(project "mcu"
+				(path "/b17ddd41-b910-4f09-a62f-46566a666def"
+					(reference "C?")
+					(unit 1)
+				)
+			)
 		)
 	)
@@
 				)
 			)
+			(project "mcu"
+				(path "/b17ddd41-b910-4f09-a62f-46566a666def"
+					(reference "CON?")
+					(unit 1)
+				)
+			)
 		)
 	)
@@
 				(path "/12cc2a67-9b1c-41e4-828f-9c2a8df6bb35/8c6fba78-5fd4-419a-8456-de6c668aaabc"
 					(reference "#PWR013")
+					(unit 1)
+				)
+			)
+			(project "mcu"
+				(path "/b17ddd41-b910-4f09-a62f-46566a666def"
+					(reference "#PWR?")
 					(unit 1)
 				)
@@
 				)
 			)
+			(project "mcu"
+				(path "/b17ddd41-b910-4f09-a62f-46566a666def"
+					(reference "C?")
+					(unit 1)
+				)
+			)
 		)
 	)
@@
 				)
 			)
+			(project "mcu"
+				(path "/b17ddd41-b910-4f09-a62f-46566a666def"
+					(reference "#PWR?")
+					(unit 1)
+				)
+			)
 		)
 	)
@@
 				)
 			)
+			(project "mcu"
+				(path "/b17ddd41-b910-4f09-a62f-46566a666def"
+					(reference "R?")
+					(unit 1)
+				)
+			)
 		)
 	)
@@
 				)
 			)
-		)
-	)
+			(project "mcu"
+				(path "/b17ddd41-b910-4f09-a62f-46566a666def"
+					(reference "#PWR?")
+					(unit 1)
+				)
+			)
+		)
+	)
+	(sheet_instances
+		(path "/"
+			(page "1")
+		)
+	)
+	(embedded_fonts no)
 )

Commit message: Port firmware to ESP32-C3-MINI-1 and replace mDNS with UDP discovery
Hardware migration (new shield revision, integrated ESP32-C3-MINI-1-N4):
- sdkconfig target esp32s3 -> esp32c3
- LED_GPIO 48 -> 7 (WS2812B-2020 on LED_CTRL / IO7)
- Implement rail-voltage sense via ADC1_CH3 (IO3), dividing R9/R10
- Schematic sheet titles "MCU (ESP32-S3-DevKitC)" -> "MCU (ESP32-C3-MINI-1)"

Replace mDNS with custom UDP discovery beacon (port 55502, 5s interval):
- mdns_hostname_set() hangs indefinitely on this board unless USB is
  attached; the managed espressif/mdns component's service_add paths
  require the main hostname, which only hostname_set() can set, so
  delegated-hostname workarounds hit the same catch-22.
- New discovery.c emits a JSON UDP broadcast the control software can
  pick up independent of router multicast / IGMP policies.
- Wire format documented in docs/discovery-protocol.md.

status_led: add set_rgb / flash_rgb / clear_override API for runtime
indicators (Modbus TCP connect white-flash, WiFi-drop orange).

Co-Authored-By: Claude Opus 4.7 (1M context) <noreply@anthropic.com>
Other:
- title: MCU (ESP32-S3-DevKitC) -> MCU (ESP32-C3-MINI-1)
Changed lines of the file:
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@@
 	(paper "A4")
 	(title_block
-		(title "MCU (ESP32-S3-DevKitC)")
+		(title "MCU (ESP32-C3-MINI-1)")
 		(date "2026-02-21")
 		(rev "1")
