File: hw/traincontrol-shield/traincontrol-shield.kicad_sch (KiCad schematic)
At the start: 6 parts, among them CON1 ConnectionPad, CON2 ConnectionPad, CON3 ConnectionPad, CON4 ConnectionPad, J1 USB_B_Micro

Commit message: Update BOM, docs, and JLCPCB outputs to match current schematics
- Update BOM.md with JLCPCB LCSC part numbers for all components
- Generate JLCPCB BOM and CPL files for PCBA ordering
- Update docs and README to reflect component changes (BAT54S/SS34
  rectification, BT134W-600E TRIACs, EL357N optocoupler, ESP32-C3)
- Suppress ERC warnings for unspecified pin connections in project settings

Co-Authored-By: Claude Opus 4.6 <noreply@anthropic.com>
Parts:
- added H1: MountingHole_Pad, MountingHole:MountingHole_2.2mm_M2_Pad, symbol Mechanical:MountingHole_Pad
Connections:
- net AC_RTN: now also H1.1
Changed lines of the file:
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@@
+	)
+	(junction
+		(at 161.29 111.76)
+		(diameter 0)
+		(color 0 0 0 0)
 	)
 	(junction
@@
 	(wire
 		(pts
-			(xy 157.48 111.76) (xy 165.1 111.76)
+			(xy 157.48 111.76) (xy 161.29 111.76)
 		)
 		(stroke
@@
 	(wire
 		(pts
+			(xy 161.29 111.76) (xy 161.29 119.38)
+		)
+		(stroke
+			(width 0)
+			(type default)
+		)
+	)
+	(wire
+		(pts
 			(xy 80 33) (xy 87.62 33)
 		)
@@
 	(wire
 		(pts
+			(xy 165.1 119.38) (xy 161.29 119.38)
+		)
+		(stroke
+			(width 0)
+			(type default)
+		)
+	)
+	(wire
+		(pts
 			(xy 252.73 69.85) (xy 252.73 71.12)
 		)
@@
 			(width 0)
 			(type default)
+		)
+	)
+	(wire
+		(pts
+			(xy 161.29 111.76) (xy 165.1 111.76)
+		)
+		(stroke
+			(width 0)
+			(type solid)
 		)
 	)
@@
 					(unit 1)
 				)
+			)
+		)
+	)
+	(symbol
+		(lib_id "Mechanical:MountingHole_Pad")
+		(at 167.64 119.38 270)
+		(unit 1)
+		(exclude_from_sim no)
+		(in_bom no)
+		(on_board yes)
+		(dnp no)
+		(fields_autoplaced yes)
+		(property "Reference" "H1"
+			(at 171.45 118.1099 90)
+			(effects
+				(font
+					(size 1.27 1.27)
+				)
+				(justify left)
+			)
+		)
+		(property "Value" "MountingHole_Pad"
+			(at 171.45 120.6499 90)
+			(effects
+				(font
+					(size 1.27 1.27)
+				)
+				(justify left)
+			)
+		)
+		(property "Footprint" "MountingHole:MountingHole_2.2mm_M2_Pad"
+			(at 167.64 119.38 0)
+			(effects
+				(font
+					(size 1.27 1.27)
+				)
+				(hide yes)
+			)
+		)
+		(property "Datasheet" "~"
+			(at 167.64 119.38 0)
+			(effects
+				(font
+					(size 1.27 1.27)
+				)
+				(hide yes)
+			)
+		)
+		(property "Description" "Mounting Hole with connection"
+			(at 167.64 119.38 0)
+			(effects
+				(font
+					(size 1.27 1.27)
+				)
+				(hide yes)
+			)
+		)
+		(pin "1"
+		)
+		(instances
+			(project ""
+				(path "/12cc2a67-9b1c-41e4-828f-9c2a8df6bb35"
+					(reference "H1")
+					(unit 1)
+				)

Commit message: Port firmware to ESP32-C3-MINI-1 and replace mDNS with UDP discovery
Hardware migration (new shield revision, integrated ESP32-C3-MINI-1-N4):
- sdkconfig target esp32s3 -> esp32c3
- LED_GPIO 48 -> 7 (WS2812B-2020 on LED_CTRL / IO7)
- Implement rail-voltage sense via ADC1_CH3 (IO3), dividing R9/R10
- Schematic sheet titles "MCU (ESP32-S3-DevKitC)" -> "MCU (ESP32-C3-MINI-1)"

Replace mDNS with custom UDP discovery beacon (port 55502, 5s interval):
- mdns_hostname_set() hangs indefinitely on this board unless USB is
  attached; the managed espressif/mdns component's service_add paths
  require the main hostname, which only hostname_set() can set, so
  delegated-hostname workarounds hit the same catch-22.
- New discovery.c emits a JSON UDP broadcast the control software can
  pick up independent of router multicast / IGMP policies.
- Wire format documented in docs/discovery-protocol.md.

status_led: add set_rgb / flash_rgb / clear_override API for runtime
indicators (Modbus TCP connect white-flash, WiFi-drop orange).

Co-Authored-By: Claude Opus 4.7 (1M context) <noreply@anthropic.com>
Other:
- sheet MCU (ESP32-S3-DevKitC) renamed MCU (ESP32-C3-MINI-1)
Changed lines of the file:
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@@
 			(color 255 255 255 1.0000)
 		)
-		(property "Sheetname" "MCU (ESP32-S3-DevKitC)"
+		(property "Sheetname" "MCU (ESP32-C3-MINI-1)"
 			(at 123.19 48.9584 0)
 			(effects
